Commit message: update for cadpackage

File: src/fullrobotassempackage/urdf/fullrobotassempackage.urdf (robot description, URDF)
Before this commit: robot fullrobotassempackage, 8 links, 7 joints
Links:
- removed link halfbody
- removed link leftarm
- removed link leftshoulder
- removed link leftwheel
- removed link rightarm
- removed link rightshoulder
- removed link rightwheel
- added link left_arm, mass 0.44382; collision mesh filename=package://fullrobotassempackage/meshes/left_arm.STL; visual mesh filename=package://fullrobotassempackage/meshes/left_arm.STL
- added link left_shoulder, mass 0.42814; collision mesh filename=package://fullrobotassempackage/meshes/left_shoulder.STL; visual mesh filename=package://fullrobotassempackage/meshes/left_shoulder.STL
- added link right_arm, mass 0.44382; collision mesh filename=package://fullrobotassempackage/meshes/right_arm.STL; visual mesh filename=package://fullrobotassempackage/meshes/right_arm.STL
- added link right_shoulder, mass 0.42814; collision mesh filename=package://fullrobotassempackage/meshes/right_shoulder.STL; visual mesh filename=package://fullrobotassempackage/meshes/right_shoulder.STL
- added link upper_body, mass 1.0125; collision mesh filename=package://fullrobotassempackage/meshes/upper_body.STL; visual mesh filename=package://fullrobotassempackage/meshes/upper_body.STL
- added link wheel_left_link, mass 0.05056; collision mesh filename=package://fullrobotassempackage/meshes/wheel_left_link.STL; visual mesh filename=package://fullrobotassempackage/meshes/wheel_left_link.STL
- added link wheel_right_link, mass 0.05056; collision mesh filename=package://fullrobotassempackage/meshes/wheel_right_link.STL; visual mesh filename=package://fullrobotassempackage/meshes/wheel_right_link.STL
- link base_link: mass 1.5842 -> 1.6424
Joints:
- removed joint armleft
- removed joint armright
- removed joint shoulderleft
- removed joint shoulderright
- removed joint upperbody
- removed joint wheelright
- added joint halfbody: type prismatic, parent base_link, child upper_body, origin xyz=0.20973 0.15434 -0.25626 rpy=3.1416 0 3.1416, axis 1 0 0, limit lower=0 upper=0.5 effort=50 velocity=0.0384
- added joint leftarm: type revolute, parent base_link, child left_arm, origin xyz=-0.20132 0.16721 -0.32659 rpy=0 -0.24449 0, axis 0 0 1, limit lower=0 upper=3.1416 effort=1.1 velocity=7.5
- added joint leftshoulder: type revolute, parent base_link, child left_shoulder, origin xyz=-0.23881 0.17058 -0.37379 rpy=0.0013991 0 0, axis 0 1 0, limit lower=0 upper=3.1416 effort=1.1 velocity=7.5
- added joint rightarm: type revolute, parent base_link, child right_arm, origin xyz=-0.39947 0.057493 -0.34727 rpy=0.057249 -0.23782 -0.23863, axis 0 0 1, limit lower=0 upper=3.1416 effort=1.1 velocity=7.5
- added joint rightshoulder: type revolute, parent base_link, child right_shoulder, origin xyz=-0.23881 0.17058 -0.37379 rpy=0 -0.021027 -3.1416, axis 0 1 0, limit lower=0 upper=3.1416 effort=1.1 velocity=7.5
- added joint rightwheel: type continuous, parent base_link, child wheel_right_link, origin xyz=0.18581 0.18863 0.30417 rpy=0 0 -3.1416, axis 0 1 0, limit lower=0 upper=0 effort=2 velocity=11.519
- joint wheelleft: axis 0 0 1 -> 0 1 0; child leftwheel -> wheel_left_link; origin xyz=0.25099 0.11429 -0.29423 rpy=-0.032213 0.080117 -2.0092 -> xyz=0.18581 0.18863 0.30417 rpy=0 0 0
