Commit message: update for cadupdate 3:56PM

File: src/fullrobotassem/urdf/fullrobotassem.urdf (robot description, URDF)
Before this commit: robot fullrobotassempackage, 8 links, 7 joints
Links:
- removed link wheel_left_link
- removed link wheel_right_link
- added link left_wheel, mass 0.05056; collision mesh filename=package://fullrobotassem/meshes/left_wheel.STL; visual mesh filename=package://fullrobotassem/meshes/left_wheel.STL
- added link right_wheel, mass 0.05056; collision mesh filename=package://fullrobotassem/meshes/right_wheel.STL; visual mesh filename=package://fullrobotassem/meshes/right_wheel.STL
- link base_link: geometry collision mesh filename=package://fullrobotassem/meshes/base_link.STL; visual mesh filename=package://fullrobotassem/meshes/base_link.STL
- link left_arm: geometry collision mesh filename=package://fullrobotassem/meshes/left_arm.STL; visual mesh filename=package://fullrobotassem/meshes/left_arm.STL
- link left_shoulder: geometry collision mesh filename=package://fullrobotassem/meshes/left_shoulder.STL; visual mesh filename=package://fullrobotassem/meshes/left_shoulder.STL
- link right_arm: geometry collision mesh filename=package://fullrobotassem/meshes/right_arm.STL; visual mesh filename=package://fullrobotassem/meshes/right_arm.STL
- link right_shoulder: mass 0.42814 -> 0.42793; geometry collision mesh filename=package://fullrobotassem/meshes/right_shoulder.STL; visual mesh filename=package://fullrobotassem/meshes/right_shoulder.STL
- link upper_body: geometry collision mesh filename=package://fullrobotassem/meshes/upper_body.STL; visual mesh filename=package://fullrobotassem/meshes/upper_body.STL
Joints:
- removed joint halfbody
- removed joint rightarm
- removed joint wheelleft
- added joint leftwheel: type continuous, parent base_link, child left_wheel, origin xyz=0.049203 0.05815 -0.14938 rpy=3.1416 0 -3.1416, axis 0 -1 0, limit lower=0 upper=0 effort=2 velocity=11.519
- added joint right_arm: type revolute, parent base_link, child right_arm, origin xyz=0.29929 0.46406 0.44707 rpy=-3.1402 0.058803 -3.1415, axis 0 0 -1, limit lower=0 upper=3.1416 effort=1.1 velocity=7.5
- added joint upperbody: type prismatic, parent base_link, child upper_body, origin xyz=-0.20973 0.15434 0.25626 rpy=0 0 0, axis 0 0 -1, limit lower=0 upper=0.5 effort=50 velocity=0.0384
- joint leftarm: axis 0 0 1 -> 0 -1 0; origin xyz=-0.20132 0.16721 -0.32659 rpy=0 -0.24449 0 -> xyz=0.28338 0.067534 0.49138 rpy=3.1416 0.24449 3.1416
- joint leftshoulder: axis 0 1 0 -> 0 -1 0; origin xyz=-0.23881 0.17058 -0.37379 rpy=0.0013991 0 0 -> xyz=0.28533 0.069834 0.49704 rpy=-3.1416 0.021027 0
- joint rightshoulder: axis 0 1 0 -> 0 -1 0; origin xyz=-0.23881 0.17058 -0.37379 rpy=0 -0.021027 -3.1416 -> xyz=0.28769 0.39622 0.49526 rpy=-0.0013994 0.021027 -2.9423E-05
- joint rightwheel: axis 0 1 0 -> 0 -1 0; child wheel_right_link -> right_wheel; origin xyz=0.18581 0.18863 0.30417 rpy=0 0 -3.1416 -> xyz=0.044232 0.41503 -0.1501 rpy=0 0 3.1416

Commit message: Update lidar and integrate model into ROS2

File: src/fullrobotassem/urdf/fullrobotassem.urdf (robot description, URDF)
Before this commit: robot fullrobotassem, 8 links, 7 joints
Links:
- added link base_footprint
- added link dummy_link
- added link lidar_link, mass 0.1; collision cylinder length=0.04 radius=0.05; visual cylinder length=0.001 radius=0.001
- link base_link: mass 1.6424 -> 15.0
Joints:
- removed joint right_arm
- added joint base_joint: type fixed, parent dummy_link, child base_link, origin xyz=0 0 0.17 rpy=0 0 0
- added joint dummy_joint: type fixed, parent base_footprint, child dummy_link, origin xyz=0 0 0 rpy=0 0 1.5708
- added joint lidar_joint: type fixed, parent base_link, child lidar_link, origin xyz=0.19 0.235 -0.02 rpy=0 0 0
- added joint right_arm_joint: type fixed, parent base_link, child right_arm, origin xyz=0 0 0 rpy=0 0 0
- joint leftarm: axis 0 -1 0 -> (none); limit lower=0 upper=3.1416 effort=1.1 velocity=7.5 -> (none); origin xyz=0.28338 0.067534 0.49138 rpy=3.1416 0.24449 3.1416 -> xyz=0 0 0 rpy=0 0 0; type revolute -> fixed
- joint leftshoulder: axis 0 -1 0 -> (none); limit lower=0 upper=3.1416 effort=1.1 velocity=7.5 -> (none); origin xyz=0.28533 0.069834 0.49704 rpy=-3.1416 0.021027 0 -> xyz=0 0 0 rpy=0 0 0; type revolute -> fixed
- joint leftwheel: axis 0 -1 0 -> (none); limit lower=0 upper=0 effort=2 velocity=11.519 -> (none); origin xyz=0.049203 0.05815 -0.14938 rpy=3.1416 0 -3.1416 -> xyz=0 0 0 rpy=0 0 0; type continuous -> fixed
- joint rightshoulder: axis 0 -1 0 -> (none); limit lower=0 upper=3.1416 effort=1.1 velocity=7.5 -> (none); origin xyz=0.28769 0.39622 0.49526 rpy=-0.0013994 0.021027 -2.9423E-05 -> xyz=0 0 0 rpy=0 0 0; type revolute -> fixed
- joint rightwheel: axis 0 -1 0 -> (none); limit lower=0 upper=0 effort=2 velocity=11.519 -> (none); origin xyz=0.044232 0.41503 -0.1501 rpy=0 0 3.1416 -> xyz=0 0 0 rpy=0 0 0; type continuous -> fixed
- joint upperbody: axis 0 0 -1 -> (none); limit lower=0 upper=0.5 effort=50 velocity=0.0384 -> (none); origin xyz=-0.20973 0.15434 0.25626 rpy=0 0 0 -> xyz=0 0 0 rpy=0 0 0; type prismatic -> fixed

Commit message: Fixed wheels coordinate issue, applied Friction and Grip for Robot

File: src/fullrobotassem/urdf/fullrobotassem.urdf (robot description, URDF)
Before this commit: robot fullrobotassem, 11 links, 10 joints
Links:
- added link caster_link, mass 0.05; collision sphere radius=0.02; visual sphere radius=0.02
- link base_link: mass 15.0 -> 2.99
- link left_wheel: geometry collision cylinder length=0.026 radius=0.03; visual mesh filename=package://fullrobotassem/meshes/left_wheel.STL
- link right_wheel: geometry collision cylinder length=0.026 radius=0.03; visual mesh filename=package://fullrobotassem/meshes/right_wheel.STL
Joints:
- added joint caster_joint: type fixed, parent base_link, child caster_link, origin xyz=0.30 0.2365 -0.159269 rpy=0 0 0
- joint base_joint: origin xyz=0 0 0.17 rpy=0 0 0 -> xyz=0 0 0.17626923 rpy=0 0 0
- joint leftwheel: axis (none) -> 0 1 0; limit (none) -> effort=0.3 velocity=11.52; origin xyz=0 0 0 rpy=0 0 0 -> xyz=0.046589 0.416034 -0.149269 rpy=0 0 0; type fixed -> continuous
- joint rightwheel: axis (none) -> 0 1 0; limit (none) -> effort=0.3 velocity=11.52; origin xyz=0 0 0 rpy=0 0 0 -> xyz=0.046589 0.057034 -0.149269 rpy=0 0 0; type fixed -> continuous

Commit message: Updated Slam toolbox and map drawing completed

File: src/fullrobotassem/urdf/fullrobotassem.urdf (robot description, URDF)
Before this commit: robot fullrobotassem, 12 links, 11 joints
Links:
- removed link dummy_link
Joints:
- removed joint dummy_joint
- joint base_joint: origin xyz=0 0 0.17626923 rpy=0 0 0 -> xyz=-0.046589 -0.236534 0.17626923 rpy=0 0 0; parent dummy_link -> base_footprint

Commit message: updated Nav2 for navigation in maze 2

File: src/fullrobotassem/urdf/fullrobotassem.urdf (robot description, URDF)
Before this commit: robot fullrobotassem, 11 links, 10 joints
Joints:
- joint leftwheel: limit effort=0.3 velocity=11.52 -> effort=5 velocity=11.52
- joint rightwheel: limit effort=0.3 velocity=11.52 -> effort=5 velocity=11.52
